File: BuzzGloveKiCad.kicad_sch (KiCad schematic)
At the start: 30 parts, among them J1 +5V, J2 8P8C, J3 GND, Q1 PN2222, Q2 PN2222, Q3 PN2222, Q4 PN2222, Q5 PN2222, Q6 PN2222

Commit message: Save version 25.04.14
Parts:
- C1: footprint Capacitor_THT:C_Radial_D6.3mm_H7.0mm_P2.50mm -> Capacitor_THT:CP_Radial_D6.3mm_P2.50mm
- J2: footprint Connector_RJ:RJ45_Amphenol_54602-x08_Horizontal -> BuzzGloveFootprints:AMPHENOL_54602-908LF
Changed lines of the file:
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@@
 			)
 		)
-		(property "Footprint" "Capacitor_THT:C_Radial_D6.3mm_H7.0mm_P2.50mm"
+		(property "Footprint" "Capacitor_THT:CP_Radial_D6.3mm_P2.50mm"
 			(at 55.88 69.85 0)
 			(effects
@@
 			)
 		)
-		(property "Footprint" "Connector_RJ:RJ45_Amphenol_54602-x08_Horizontal"
+		(property "Footprint" "BuzzGloveFootprints:AMPHENOL_54602-908LF"
 			(at 40.64 136.525 90)
 			(effects

Commit message: This is what was shipped to pcbway today.
Small silk screen changes.
Parts:
- added J4: Power, Connector_JST:JST_PH_B2B-PH-K_1x02_P2.00mm_Vertical, symbol Connector_Generic:Conn_01x02
Connections:
- net +5V: now also J4.1 (Pin_1)
- net GND: now also J4.2 (Pin_2)
Other:
- company: (none) -> FRC3620 - Average Joes
- title: (none) -> BuzzGloves
Changed lines of the file:
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@@
 	(generator_version "9.0")
 	(paper "USLetter")
+	(title_block
+		(title "BuzzGloves")
+		(date "2025-06-24")
+		(rev "2025.06.23")
+		(company "FRC3620 - Average Joes")
+	)
 	(junction
 		(at 196.85 83.82)
@@
 	)
 	(junction
+		(at 45.72 78.74)
+		(diameter 0)
+		(color 0 0 0 0)
+	)
+	(junction
 		(at 205.74 139.7)
 		(diameter 0)
@@
 	(wire
 		(pts
+			(xy 39.37 67.31) (xy 45.72 67.31)
+		)
+		(stroke
+			(width 0)
+			(type default)
+		)
+	)
+	(wire
+		(pts
 			(xy 196.85 129.54) (xy 198.12 129.54)
 		)
@@
 	(wire
 		(pts
+			(xy 39.37 69.85) (xy 45.72 69.85)
+		)
+		(stroke
+			(width 0)
+			(type default)
+		)
+	)
+	(wire
+		(pts
 			(xy 243.84 121.92) (xy 243.84 124.46)
 		)
@@
 	(wire
 		(pts
-			(xy 39.37 78.74) (xy 55.88 78.74)
+			(xy 39.37 78.74) (xy 45.72 78.74)
 		)
 		(stroke
@@
 	(wire
 		(pts
+			(xy 45.72 69.85) (xy 45.72 78.74)
+		)
+		(stroke
+			(width 0)
+			(type default)
+		)
+	)
+	(wire
+		(pts
 			(xy 167.64 67.31) (xy 167.64 68.58)
 		)
@@
 	(wire
 		(pts
+			(xy 45.72 67.31) (xy 45.72 58.42)
+		)
+		(stroke
+			(width 0)
+			(type default)
+		)
+	)
+	(wire
+		(pts
 			(xy 196.85 83.82) (xy 198.12 83.82)
 		)
@@
 		)
 	)
+	(wire
+		(pts
+			(xy 45.72 78.74) (xy 55.88 78.74)
+		)
+		(stroke
+			(width 0)
+			(type default)
+		)
+	)
 	(label "Pico Power"
 		(at 100.33 67.31 0)
@@
 	)
 	(symbol
+		(lib_id "Connector_Generic:Conn_01x02")
+		(at 34.29 67.31 0)
+		(mirror y)
+		(unit 1)
+		(exclude_from_sim no)
+		(in_bom yes)
+		(on_board yes)
+		(dnp no)
+		(property "Reference" "J4"
+			(at 31.75 67.3099 0)
+			(effects
+				(font
+					(size 1.27 1.27)
+				)
+				(justify left)
+				(hide yes)
+			)
+		)
+		(property "Value" "Power"
+			(at 31.75 69.8499 0)
+			(effects
+				(font
+					(size 1.27 1.27)
+				)
+				(justify left)
+			)
+		)
+		(property "Footprint" "Connector_JST:JST_PH_B2B-PH-K_1x02_P2.00mm_Vertical"
+			(at 34.29 67.31 0)
+			(effects
+				(font
+					(size 1.27 1.27)
+				)
+				(hide yes)
+			)
+		)
+		(property "Datasheet" "~"
+			(at 34.29 67.31 0)
+			(effects
+				(font
+					(size 1.27 1.27)
+				)
+				(hide yes)
+			)
+		)
+		(property "Description" "Generic connector, single row, 01x02, script generated (kicad-library-utils/schlib/autogen/connector/)"
+			(at 34.29 67.31 0)
+			(effects
+				(font
+					(size 1.27 1.27)
+				)
+				(hide yes)
+			)
+		)
+		(pin "1"
+		)
+		(pin "2"
+		)
+		(instances
+			(project ""
+				(path "/96e18a86-4139-49e1-85cc-a3b99f8c401d"
+					(reference "J4")
+					(unit 1)
+				)
+			)
+		)
+	)
+	(symbol
 		(lib_id "Device:R_US")
 		(at 229.87 83.82 270)
@@
 	)
 	(embedded_fonts no)
+	(embedded_files
+		(file
+			(name "frc3620.kicad_wks")
+			(type worksheet)
+			(data |KLUv/WB5CMUTAEZdXCEAtxsWHGS5ac4JWli9n5JTOUAZRYkn5HXQcxNVVbcAEAFSAEsAVQD/uBPx
+				fzw2T9rXejIXbt9x0GBROfvznyX5taDBkrT9ZMcv+RcAgIBAFL2PU17VVtnPN1CsOuPnsl/3GBiU
+				UkSdtS+2Y/ZRARAQjCHS9nGeDRUCJf/urYmwak/LVMretf2ci94z+83Ye7BnzyrkYbBrB99+++f7
+				uyKcua76r4ch9uacsnbt73qtEyFn7UtR5aS0P3M/VlV7yN33PIc4I78wGFVHqEz0NSmlomEu2WZ7
+				YA4tgiJY0pJWT0ovqegFI5VlsMeWaTAYDUXohj/3yDmbsv91r00d+6MIZNWmmKlaPbuumxRRAPzF
+				HdpW7RGLFa36AwGBQVGvy3Q5McSOhFxwKJhlUnFMxSUthExMMEom0SAW4lmQe9uG2nUhJ80kGS0D
+				vs1UWuln+90/mMEhNfi0qp8LM+50dpGzXDILZvGTxXwg7jpRtU12CW2g4TSnHJoSEUmSJB1gRKQG
+				qxvfEWMwPuTpCXcvk63bpXvJL4vxOU1sBhC7gLnxpYlheHkdzpeBNkXADDan5j6RUHL6RNnzXfLD
+				JD6Uvz2EFGJi1rANwb6DQx75ji3ic3bK80QHDHF+WuiJxsZYKhy0ZMrTaBj0Uo5isnacupIH3J95
+				Wn5sM3/IHtVhiIY8+aC5sjU3+WwslwjWOVrWUhwUxGgcpz3oV+LNCR7Q2+M9VisIMolZjXVnvvQE
+				akMdnzbBgGarJqUH3SLCCmNQkGedmeCQJGaTQOfVRyEq57PbILlTZQcJ7c3Lb0eGn+Idwz4F2vR8
+				/Vrr/3F8RP1kuQP+GJgq|
+			)
+			(checksum "4FC45D2661D23489CE359C90BCD367E1")
+		)
+	)
 )
