File: BuzzGloveKiCad.kicad_pcb (KiCad board)
At the start: 2 copper layers, 67.3 x 80.2 mm, 33 parts, among them J1 +5V, J2 8P8C, J3 GND, Q1 PN2222, Q2 PN2222, Q3 PN2222, Q4 PN2222, Q5 PN2222, Q6 PN2222

Commit message: Save version 25.04.14
Parts:
- removed the REF** at (118.1, 62.9)
- removed the REF** at (174.0, 131.4)
- added REF**: MountingHole_3.2mm_M3, MountingHole:MountingHole_3.2mm_M3, F.Cu at (172.7, 128.3)
- added REF**: MountingHole_3.2mm_M3, MountingHole:MountingHole_3.2mm_M3, F.Cu at (119.4, 63.5)
- C1: footprint Capacitor_THT:C_Radial_D6.3mm_H7.0mm_P2.50mm -> Capacitor_THT:CP_Radial_D6.3mm_P2.50mm
- J2: footprint Connector_RJ:RJ45_Amphenol_54602-x08_Horizontal -> BuzzGloveFootprints:AMPHENOL_54602-908LF
- moved G*** 64.8 mm to (118.1, 83.5), turned to -90 degrees
- moved C1 34.1 mm to (158.2, 119.4), turned to 0 degrees
- moved J2 7.69 mm to (146.1, 129.5)
- moved J3 7.20 mm to (120.0, 125.7)
- moved J1 6.11 mm to (133.3, 125.7)
- moved Q4 1.91 mm to (130.2, 115.5)
- moved Q5 1.91 mm to (125.7, 121.8)
- moved Q6 1.91 mm to (121.3, 115.5)
- moved Q1 0.36 mm to (161.9, 109.9)
Routing:
- net +5V: track 145.3 -> 150.9 mm
- net X1: track 18.7 -> 20.6 mm
- net /DummyLoad: track 10.2 -> 11.6 mm
- net X5: track 10.4 -> 11.6 mm
- net X4: track 11.6 -> 12.9 mm
- net M5: track 35.7 -> 34.5 mm
- net M4: track 25.0 -> 23.8 mm
- net X3: track 27.2 -> 28.4 mm
- net X6: track 10.5 -> 11.6 mm
- net X2: track 31.0 -> 32.0 mm
- net Net-(Q6-B): track 46.8 -> 47.7 mm
- net Net-(Q5-B): track 35.7 -> 36.5 mm
- net Net-(Q4-B): track 38.5 -> 39.3 mm
Other:
- board size 67.3 x 80.2 mm -> 66 x 77.4 mm
- board text added: "EF 2025.04.14"
- board text removed: "EF 2025.04.04"

Commit message: This is what was shipped to pcbway today.
Small silk screen changes.
Parts:
- added J4: Power, Connector_JST:JST_PH_B2B-PH-K_1x02_P2.00mm_Vertical, F.Cu at (160.9, 128.4)
- R13: value 1kΩ -> (1kΩ)
- R14: value 10kΩ -> (10kΩ)
- R15: value 100Ω -> (100Ω)
- moved J2 1.32 mm to (144.8, 129.5)
- moved J3 1.27 mm to (118.7, 125.7)
- moved J1 0.63 mm to (132.7, 125.7)
- renumbered Q6 to (Q6)
Routing:
- net +5V: track 150.9 -> 164.4 mm
- net M5: track 34.5 -> 32.5 mm
- net M4: track 23.8 -> 21.8 mm
- net M2: track 36.3 -> 37.6 mm
- net M1: track 31.6 -> 32.2 mm
- net M3: track 46.6 -> 47.1 mm
Other:
- board text added: "EF 2025.06.23"
- board text removed: "EF 2025.04.14"

Commit message: Print color codes on silkscreen.
Other:
- board text added: "1kΩ = BRN BLK RED 10KΩ = BRN BLK ORG"
- board text added: "EF 2025.08.19"
- board text removed: "EF 2025.06.23"
Changed lines of the file:
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@@
 		(layer "Edge.Cuts")
 	)
-	(gr_text "EF 2025.06.23"
+	(gr_text "1kΩ = BRN BLK RED\n10KΩ = BRN BLK ORG"
+		(at 162.56 90.805 90)
+		(layer "F.SilkS")
+		(effects
+			(font
+				(size 1 1)
+				(thickness 0.1)
+			)
+			(justify left bottom)
+		)
+	)
+	(gr_text "EF 2025.08.19"
 		(at 117.475 130.81 0)
 		(layer "F.SilkS")
